File: kicad/lcd.kicad_sch (KiCad schematic)
At the start: 1 part, among them J1 Conn_01x08_Pin

Commit message: adjustments to design on kicad
Parts:
- J1: footprint (none) -> Connector_PinHeader_2.54mm:PinHeader_1x08_P2.54mm_Vertical
Changed lines of the file:
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@@
       (effects (font (size 1.27 1.27)))
     )
-    (property "Footprint" "" (at 124.46 86.36 0)
+    (property "Footprint" "Connector_PinHeader_2.54mm:PinHeader_1x08_P2.54mm_Vertical" (at 124.46 86.36 0)
       (effects (font (size 1.27 1.27)) hide)
     )

Commit message: completed board layout and passed drc
Connections:
- net LCD_CS: now also J1.7 (Pin_7)
- net LCD_DC: now also J1.6 (Pin_6)
- net LCD_RES: now also J1.5 (Pin_5)
- net LCD_SCL: now also J1.3 (Pin_3)
- net LCD_SDA: now also J1.4 (Pin_4)

Commit message: routed pcb, only bom left to do
Parts:
- J1: now not fitted
Changed lines of the file:
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@@
 		(in_bom yes)
 		(on_board yes)
-		(dnp no)
+		(dnp yes)
 		(fields_autoplaced yes)
 		(property "Reference" "J1"
@@
 			)
 		)
-		(property "Description" ""
+		(property "Description" "Generic connector, single row, 01x08, script generated"
 			(at 124.46 86.36 0)
 			(effects
@@
 		)
 		(property "Value" "GND"
-			(at 133.35 78.74 90)
+			(at 133.35 78.7399 90)
 			(effects
 				(font
@@
 			)
 		)
-		(property "Description" ""
+		(property "Description" "Power symbol creates a global label with name \"GND\" , ground"
 			(at 129.54 78.74 0)
 			(effects
@@
 		)
 		(property "Value" "+3V3"
-			(at 143.51 73.66 0)
+			(at 146.05 77.4699 0)
 			(effects
 				(font
 					(size 1.27 1.27)
 				)
+				(justify left)
 			)
 		)
@@
 			)
 		)
-		(property "Description" ""
+		(property "Description" "Power symbol creates a global label with name \"+3V3\""
 			(at 143.51 78.74 0)
 			(effects
