File: kicad/project.kicad_pcb (KiCad board)
At the start: 2 copper layers, 58.4 x 58.4 mm, 22 parts, among them J1 Conn_01x08_Pin, J2 PiZeroW_Bottom_Mount

Commit message: completed board layout and passed drc
Parts:
- added REF**: MountingHole_2.7mm_M2.5, MountingHole:MountingHole_2.7mm_M2.5, F.Cu at (130.3, 43.9)
- added REF**: MountingHole_2.7mm_M2.5, MountingHole:MountingHole_2.7mm_M2.5, F.Cu at (77.3, 49.9)
- added REF**: MountingHole_2.7mm_M2.5, MountingHole:MountingHole_2.7mm_M2.5, F.Cu at (107.3, 49.9)
- added REF**: MountingHole_2.7mm_M2.5, MountingHole:MountingHole_2.7mm_M2.5, F.Cu at (107.3, 101.9)
- added REF**: MountingHole_2.7mm_M2.5, MountingHole:MountingHole_2.7mm_M2.5, F.Cu at (130.3, 101.9)
- added REF**: MountingHole_2.7mm_M2.5, MountingHole:MountingHole_2.7mm_M2.5, F.Cu at (107.3, 43.9)
- added REF**: MountingHole_2.7mm_M2.5, MountingHole:MountingHole_2.7mm_M2.5, F.Cu at (77.3, 101.9)
- moved R10 7.25 mm to (115.3, 84.2)
- moved J1 6.07 mm to (101.2, 102.4)
- moved R9 5.83 mm to (115.4, 77.2)
- moved R8 4.66 mm to (115.3, 70.2)
- moved PWR1 3.21 mm to (116.7, 50.0)
- moved APP_3 3.09 mm to (115.3, 81.6)
- moved R6 3.09 mm to (116.7, 53.5)
- moved R3 2.80 mm to (122.0, 91.0)
- moved SW_APP_3 2.78 mm to (121.8, 81.6)
- moved LAN1 2.49 mm to (123.4, 50.0)
- moved R7 2.34 mm to (123.4, 53.5)
- moved R2 2.31 mm to (122.0, 88.0)
- moved R1 1.82 mm to (122.0, 85.0)
- moved SW_APP_2 1.61 mm to (121.8, 75.3)
- moved R4 1.36 mm to (114.6, 63.0)
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Connections:
- J1 pad 3: unconnected-(J1-Pin_3-Pad3) -> /LCD_Display/LCD_SCL
- J1 pad 4: unconnected-(J1-Pin_4-Pad4) -> /LCD_Display/LCD_SDA
- J1 pad 5: unconnected-(J1-Pin_5-Pad5) -> /LCD_Display/LCD_RES
- J1 pad 6: unconnected-(J1-Pin_6-Pad6) -> /LCD_Display/LCD_DC
- J1 pad 7: unconnected-(J1-Pin_7-Pad7) -> /LCD_Display/LCD_CS
Other:
- board size 58.4 x 58.4 mm -> 61 x 66.1 mm

Commit message: routed pcb, only bom left to do
Parts:
- moved R1 16.8 mm to (126.0, 68.7), turned to -90 degrees
- moved R2 13.2 mm to (126.0, 75.4), turned to -90 degrees
- moved R3 10.2 mm to (126.0, 81.6), turned to -90 degrees
- turned APP_1 to 180 degrees
- turned APP_2 to 180 degrees
- turned APP_3 to 180 degrees
- turned R10 to 180 degrees
- turned R8 to 180 degrees
- turned R9 to 180 degrees
- renumbered REF** to H1, REF** to H2, REF** to H3, REF** to H4/7, REF** to H5, REF** to H6, REF** to H8
Connections:
- J2 pad 14: unconnected-(J2-GND-Pad14) -> GND
- J2 pad 17: unconnected-(J2-3V3-Pad17) -> +3V3
- J2 pad 20: unconnected-(J2-GND-Pad20) -> GND
- J2 pad 25: unconnected-(J2-GND-Pad25) -> GND
- J2 pad 30: unconnected-(J2-GND-Pad30) -> GND
- J2 pad 34: unconnected-(J2-GND-Pad34) -> GND
- J2 pad 39: unconnected-(J2-GND-Pad39) -> GND
- J2 pad 9: unconnected-(J2-GND-Pad9) -> GND
Routing:
- net +3V3: track 0.00 -> 188.5 mm
- net /LCD_Display/LCD_CS: track 0.00 -> 72.1 mm
- net /LCD_Display/LCD_DC: track 0.00 -> 68.6 mm
- net /LCD_Display/LCD_RES: track 0.00 -> 64.6 mm
- net /LED_Panel/LAN_LED: track 0.00 -> 57.1 mm
- net /LCD_Display/LCD_SDA: track 0.00 -> 55.8 mm
- net /LCD_Display/LCD_SCL: track 0.00 -> 47.0 mm
- net /LED_Panel/APP_LED_1: track 0.00 -> 41.0 mm
- net /LED_Panel/APP_LED_2: track 0.00 -> 40.5 mm
- net /LED_Panel/APP_LED_3: track 0.00 -> 39.1 mm
- net /Control_Panel/TGL_APP_1: track 0.00 -> 38.9 mm
- net /Control_Panel/EV_BAT_P: track 0.00 -> 27.9 mm
- net GND: track 0.00 -> 27.2 mm, vias 0 -> 10
- net /Control_Panel/EV_BAT_N: track 0.00 -> 26.1 mm
- net /Control_Panel/TGL_APP_2: track 0.00 -> 17.4 mm
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- added copper zone on B.Cu, net GND
Other:
- board size 61 x 66.1 mm -> 61.6 x 66.1 mm
