File: kicad/control_panel.kicad_sch (KiCad schematic)
At the start: 8 parts, among them SW1 SW_Push, SW2 SW_Push, SW3 SW_Push

Commit message: developed proper schematic in KiCad along with supporting firmware. code still doesnt gracefully handle all errors but it now does for ureq (network) errors, turning the LAN light off but not ejecting
Parts:
- removed R5: R_Variable, symbol Device:R_Variable
- added R5: 10k, symbol Device:R
- added SW4, SW5: SW_Push, symbol Switch:SW_Push
- R1, R2, R3, R4: value R -> 10k
Connections:
- net +3V3: now also R5.1
- net GND: now also SW4.1, SW5.1
- net CAR_PWR_SLD renamed EV_BAT_P
- net EV_BAT_P: now also SW4.2
- new net EV_BAT_N: R5.2, SW5.2

Commit message: adjustments to design on kicad
Parts:
- R1, R2, R3, R4, R5: footprint (none) -> Resistor_SMD:R_0603_1608Metric
- SW_APP_1: renamed from SW1; footprint (none) -> Button_Switch_SMD:SW_SPST_PTS810
- SW_APP_2: renamed from SW2; footprint (none) -> Button_Switch_SMD:SW_SPST_PTS810
- SW_APP_3: renamed from SW3; footprint (none) -> Button_Switch_SMD:SW_SPST_PTS810
- SW_EV_N1: renamed from SW5; footprint (none) -> Button_Switch_SMD:SW_SPST_PTS810
- SW_EV_P1: renamed from SW4; footprint (none) -> Button_Switch_SMD:SW_SPST_PTS810
Changed lines of the file:
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@@
       (effects (font (size 1.27 1.27)) (justify left))
     )
-    (property "Footprint" "" (at 66.802 58.42 90)
+    (property "Footprint" "Resistor_SMD:R_0603_1608Metric" (at 66.802 58.42 90)
       (effects (font (size 1.27 1.27)) hide)
     )
@@
       (effects (font (size 1.27 1.27)) (justify left))
     )
-    (property "Footprint" "" (at 116.332 58.42 90)
+    (property "Footprint" "Resistor_SMD:R_0603_1608Metric" (at 116.332 58.42 90)
       (effects (font (size 1.27 1.27)) hide)
     )
@@
       (effects (font (size 1.27 1.27)) (justify left))
     )
-    (property "Footprint" "" (at 99.822 58.42 90)
+    (property "Footprint" "Resistor_SMD:R_0603_1608Metric" (at 99.822 58.42 90)
       (effects (font (size 1.27 1.27)) hide)
     )
@@
   (symbol (lib_id "Switch:SW_Push") (at 101.6 74.93 90) (unit 1)
     (in_bom yes) (on_board yes) (dnp no) (fields_autoplaced)
-    (property "Reference" "SW3" (at 102.87 73.6599 90)
-      (effects (font (size 1.27 1.27)) (justify right))
-    )
-    (property "Value" "SW_Push" (at 102.87 76.1999 90)
-      (effects (font (size 1.27 1.27)) (justify right))
-    )
-    (property "Footprint" "" (at 96.52 74.93 0)
+    (property "Reference" "SW_APP_3" (at 102.87 73.66 90)
+      (effects (font (size 1.27 1.27)) (justify right))
+    )
+    (property "Value" "SW_Push" (at 102.87 76.2 90)
+      (effects (font (size 1.27 1.27)) (justify right))
+    )
+    (property "Footprint" "Button_Switch_SMD:SW_SPST_PTS810" (at 96.52 74.93 0)
       (effects (font (size 1.27 1.27)) hide)
     )
@@
       (project "project"
         (path "/9538e4ed-27e6-4c37-b989-9859dc0d49e8/619eee36-7c04-46f2-a8c0-8355d58d5928"
-          (reference "SW3") (unit 1)
+          (reference "SW_APP_3") (unit 1)
         )
       )
@@
       (effects (font (size 1.27 1.27)) (justify left))
     )
-    (property "Footprint" "" (at 83.312 58.42 90)
+    (property "Footprint" "Resistor_SMD:R_0603_1608Metric" (at 83.312 58.42 90)
       (effects (font (size 1.27 1.27)) hide)
     )
@@
   (symbol (lib_id "Switch:SW_Push") (at 68.58 74.93 90) (unit 1)
     (in_bom yes) (on_board yes) (dnp no) (fields_autoplaced)
-    (property "Reference" "SW1" (at 69.85 73.6599 90)
-      (effects (font (size 1.27 1.27)) (justify right))
-    )
-    (property "Value" "SW_Push" (at 69.85 76.1999 90)
-      (effects (font (size 1.27 1.27)) (justify right))
-    )
-    (property "Footprint" "" (at 63.5 74.93 0)
+    (property "Reference" "SW_APP_1" (at 69.85 73.66 90)
+      (effects (font (size 1.27 1.27)) (justify right))
+    )
+    (property "Value" "SW_Push" (at 69.85 76.2 90)
+      (effects (font (size 1.27 1.27)) (justify right))
+    )
+    (property "Footprint" "Button_Switch_SMD:SW_SPST_PTS810" (at 63.5 74.93 0)
       (effects (font (size 1.27 1.27)) hide)
     )
@@
       (project "project"
         (path "/9538e4ed-27e6-4c37-b989-9859dc0d49e8/619eee36-7c04-46f2-a8c0-8355d58d5928"
-          (reference "SW1") (unit 1)
+          (reference "SW_APP_1") (unit 1)
         )
       )
@@
   (symbol (lib_id "Switch:SW_Push") (at 134.62 74.93 90) (unit 1)
     (in_bom yes) (on_board yes) (dnp no) (fields_autoplaced)
-    (property "Reference" "SW5" (at 135.89 73.6599 90)
+    (property "Reference" "SW_EV_N1" (at 135.89 73.6599 90)
       (effects (font (size 1.27 1.27)) (justify right))
     )
@@
       (effects (font (size 1.27 1.27)) (justify right))
     )
-    (property "Footprint" "" (at 129.54 74.93 0)
+    (property "Footprint" "Button_Switch_SMD:SW_SPST_PTS810" (at 129.54 74.93 0)
       (effects (font (size 1.27 1.27)) hide)
     )
@@
       (project "project"
         (path "/9538e4ed-27e6-4c37-b989-9859dc0d49e8/619eee36-7c04-46f2-a8c0-8355d58d5928"
-          (reference "SW5") (unit 1)
+          (reference "SW_EV_N1") (unit 1)
         )
       )
@@
   (symbol (lib_id "Switch:SW_Push") (at 118.11 74.93 90) (unit 1)
     (in_bom yes) (on_board yes) (dnp no) (fields_autoplaced)
-    (property "Reference" "SW4" (at 119.38 73.6599 90)
-      (effects (font (size 1.27 1.27)) (justify right))
-    )
-    (property "Value" "SW_Push" (at 119.38 76.1999 90)
-      (effects (font (size 1.27 1.27)) (justify right))
-    )
-    (property "Footprint" "" (at 113.03 74.93 0)
+    (property "Reference" "SW_EV_P1" (at 119.38 73.66 90)
+      (effects (font (size 1.27 1.27)) (justify right))
+    )
+    (property "Value" "SW_Push" (at 119.38 76.2 90)
+      (effects (font (size 1.27 1.27)) (justify right))
+    )
+    (property "Footprint" "Button_Switch_SMD:SW_SPST_PTS810" (at 113.03 74.93 0)
       (effects (font (size 1.27 1.27)) hide)
     )
@@
       (project "project"
         (path "/9538e4ed-27e6-4c37-b989-9859dc0d49e8/619eee36-7c04-46f2-a8c0-8355d58d5928"
-          (reference "SW4") (unit 1)
+          (reference "SW_EV_P1") (unit 1)
         )
       )
@@
   (symbol (lib_id "power:+3V3") (at 68.58 52.07 0) (unit 1)
     (in_bom yes) (on_board yes) (dnp no) (fields_autoplaced)
-    (property "Reference" "#PWR?" (at 68.58 55.88 0)
+    (property "Reference" "#PWR0101" (at 68.58 55.88 0)
       (effects (font (size 1.27 1.27)) hide)
     )
@@
       (project "project"
         (path "/9538e4ed-27e6-4c37-b989-9859dc0d49e8/619eee36-7c04-46f2-a8c0-8355d58d5928"
-          (reference "#PWR?") (unit 1)
+          (reference "#PWR0101") (unit 1)
         )
       )
@@
   (symbol (lib_id "Switch:SW_Push") (at 85.09 74.93 90) (unit 1)
     (in_bom yes) (on_board yes) (dnp no) (fields_autoplaced)
-    (property "Reference" "SW2" (at 86.36 73.6599 90)
-      (effects (font (size 1.27 1.27)) (justify right))
-    )
-    (property "Value" "SW_Push" (at 86.36 76.1999 90)
-      (effects (font (size 1.27 1.27)) (justify right))
-    )
-    (property "Footprint" "" (at 80.01 74.93 0)
+    (property "Reference" "SW_APP_2" (at 86.36 73.66 90)
+      (effects (font (size 1.27 1.27)) (justify right))
+    )
+    (property "Value" "SW_Push" (at 86.36 76.2 90)
+      (effects (font (size 1.27 1.27)) (justify right))
+    )
+    (property "Footprint" "Button_Switch_SMD:SW_SPST_PTS810" (at 80.01 74.93 0)
       (effects (font (size 1.27 1.27)) hide)
     )
@@
       (project "project"
         (path "/9538e4ed-27e6-4c37-b989-9859dc0d49e8/619eee36-7c04-46f2-a8c0-8355d58d5928"
-          (reference "SW2") (unit 1)
+          (reference "SW_APP_2") (unit 1)
         )
       )
@@
       (effects (font (size 1.27 1.27)) (justify left))
     )
-    (property "Footprint" "" (at 132.842 58.42 90)
+    (property "Footprint" "Resistor_SMD:R_0603_1608Metric" (at 132.842 58.42 90)
       (effects (font (size 1.27 1.27)) hide)
     )
@@
   (symbol (lib_id "power:GND") (at 134.62 87.63 0) (unit 1)
     (in_bom yes) (on_board yes) (dnp no) (fields_autoplaced)
-    (property "Reference" "#PWR?" (at 134.62 93.98 0)
+    (property "Reference" "#PWR0102" (at 134.62 93.98 0)
       (effects (font (size 1.27 1.27)) hide)
     )
@@
       (project "project"
         (path "/9538e4ed-27e6-4c37-b989-9859dc0d49e8/619eee36-7c04-46f2-a8c0-8355d58d5928"
-          (reference "#PWR?") (unit 1)
-        )
-      )
+          (reference "#PWR0102") (unit 1)
+        )
+      )

Commit message: routed pcb, only bom left to do
Changed lines of the file:
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@@
 			)
 		)
-		(property "Description" ""
+		(property "Description" "Resistor"
 			(at 68.58 58.42 0)
 			(effects
@@
 		(fields_autoplaced yes)
 		(property "Reference" "R4"
-			(at 120.65 57.15 0)
+			(at 120.65 57.1499 0)
 			(effects
 				(font
@@
 		)
 		(property "Value" "10k"
-			(at 120.65 59.69 0)
+			(at 120.65 59.6899 0)
 			(effects
 				(font
@@
 			)
 		)
-		(property "Description" ""
+		(property "Description" "Resistor"
 			(at 118.11 58.42 0)
 			(effects
@@
 		(fields_autoplaced yes)
 		(property "Reference" "R3"
-			(at 104.14 57.15 0)
+			(at 104.14 57.1499 0)
 			(effects
 				(font
@@
 		)
 		(property "Value" "10k"
-			(at 104.14 59.69 0)
+			(at 104.14 59.6899 0)
 			(effects
 				(font
@@
 			)
 		)
-		(property "Description" ""
+		(property "Description" "Resistor"
 			(at 101.6 58.42 0)
 			(effects
@@
 		(fields_autoplaced yes)
 		(property "Reference" "SW_APP_3"
-			(at 102.87 73.66 90)
+			(at 102.87 73.6599 90)
 			(effects
 				(font
@@
 		)
 		(property "Value" "SW_Push"
-			(at 102.87 76.2 90)
+			(at 102.87 76.1999 90)
 			(effects
 				(font
@@
 			)
 		)
-		(property "Description" ""
+		(property "Description" "Push button switch, generic, two pins"
 			(at 101.6 74.93 0)
 			(effects
@@
 			)
 		)
-		(property "Description" ""
+		(property "Description" "Resistor"
 			(at 85.09 58.42 0)
 			(effects
@@
 		(fields_autoplaced yes)
 		(property "Reference" "SW_APP_1"
-			(at 69.85 73.66 90)
+			(at 69.85 73.6599 90)
 			(effects
 				(font
@@
 		)
 		(property "Value" "SW_Push"
-			(at 69.85 76.2 90)
+			(at 69.85 76.1999 90)
 			(effects
 				(font
@@
 			)
 		)
-		(property "Description" ""
+		(property "Description" "Push button switch, generic, two pins"
 			(at 68.58 74.93 0)
 			(effects
@@
 			)
 		)
-		(property "Description" ""
+		(property "Description" "Push button switch, generic, two pins"
 			(at 134.62 74.93 0)
 			(effects
@@
 		(fields_autoplaced yes)
 		(property "Reference" "SW_EV_P1"
-			(at 119.38 73.66 90)
+			(at 119.38 73.6599 90)
 			(effects
 				(font
@@
 		)
 		(property "Value" "SW_Push"
-			(at 119.38 76.2 90)
+			(at 119.38 76.1999 90)
 			(effects
 				(font
@@
 			)
 		)
-		(property "Description" ""
+		(property "Description" "Push button switch, generic, two pins"
 			(at 118.11 74.93 0)
 			(effects
@@
 		)
 		(property "Value" "+3V3"
-			(at 68.58 46.99 0)
-			(effects
-				(font
-					(size 1.27 1.27)
-				)
+			(at 71.12 50.7999 0)
+			(effects
+				(font
+					(size 1.27 1.27)
+				)
+				(justify left)
 			)
 		)
@@
 			)
 		)
-		(property "Description" ""
+		(property "Description" "Power symbol creates a global label with name \"+3V3\""
 			(at 68.58 52.07 0)
 			(effects
@@
 		(fields_autoplaced yes)
 		(property "Reference" "SW_APP_2"
-			(at 86.36 73.66 90)
+			(at 86.36 73.6599 90)
 			(effects
 				(font
@@
 		)
 		(property "Value" "SW_Push"
-			(at 86.36 76.2 90)
+			(at 86.36 76.1999 90)
 			(effects
 				(font
@@
 			)
 		)
-		(property "Description" ""
+		(property "Description" "Push button switch, generic, two pins"
 			(at 85.09 74.93 0)
 			(effects
@@
 		(fields_autoplaced yes)
 		(property "Reference" "R5"
-			(at 137.16 57.15 0)
+			(at 137.16 57.1499 0)
 			(effects
 				(font
@@
 		)
 		(property "Value" "10k"
-			(at 137.16 59.69 0)
+			(at 137.16 59.6899 0)
 			(effects
 				(font
@@
 			)
 		)
-		(property "Description" ""
+		(property "Description" "Resistor"
 			(at 134.62 58.42 0)
 			(effects
@@
 		)
 		(property "Value" "GND"
-			(at 134.62 92.71 0)
-			(effects
-				(font
-					(size 1.27 1.27)
-				)
+			(at 137.16 88.8999 0)
+			(effects
+				(font
+					(size 1.27 1.27)
+				)
+				(justify left)
 			)
 		)
@@
 			)
 		)
-		(property "Description" ""
+		(property "Description" "Power symbol creates a global label with name \"GND\" , ground"
 			(at 134.62 87.63 0)
 			(effects

Commit message: kicad changes
Parts:
- R1, R2, R3, R4, R5: LCSC (none) -> C98220
- SW_APP_1, SW_APP_2, SW_APP_3, SW_EV_N1, SW_EV_P1: LCSC (none) -> C139797
Changed lines of the file:
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@@
+			)
+		)
+		(property "LCSC" "C98220"
+			(at 68.58 58.42 0)
+			(effects
+				(font
+					(size 1.27 1.27)
+				)
+				(hide yes)
 			)
 		)
@@
 			)
 		)
+		(property "LCSC" "C98220"
+			(at 118.11 58.42 0)
+			(effects
+				(font
+					(size 1.27 1.27)
+				)
+				(hide yes)
+			)
+		)
 		(pin "1"
 		)
@@
 			)
 		)
+		(property "LCSC" "C98220"
+			(at 101.6 58.42 0)
+			(effects
+				(font
+					(size 1.27 1.27)
+				)
+				(hide yes)
+			)
+		)
 		(pin "1"
 		)
@@
 			)
 		)
+		(property "LCSC" "C139797"
+			(at 101.6 74.93 90)
+			(effects
+				(font
+					(size 1.27 1.27)
+				)
+				(hide yes)
+			)
+		)
 		(pin "1"
 		)
@@
 			)
 		)
+		(property "LCSC" "C98220"
+			(at 85.09 58.42 0)
+			(effects
+				(font
+					(size 1.27 1.27)
+				)
+				(hide yes)
+			)
+		)
 		(pin "1"
 		)
@@
 			)
 		)
+		(property "LCSC" "C139797"
+			(at 68.58 74.93 90)
+			(effects
+				(font
+					(size 1.27 1.27)
+				)
+				(hide yes)
+			)
+		)
 		(pin "1"
 		)
@@
 			)
 		)
+		(property "LCSC" "C139797"
+			(at 134.62 74.93 90)
+			(effects
+				(font
+					(size 1.27 1.27)
+				)
+				(hide yes)
+			)
+		)
 		(pin "1"
 		)
@@
 			)
 		)
+		(property "LCSC" "C139797"
+			(at 118.11 74.93 90)
+			(effects
+				(font
+					(size 1.27 1.27)
+				)
+				(hide yes)
+			)
+		)
 		(pin "1"
 		)
@@
 			)
 		)
+		(property "LCSC" "C139797"
+			(at 85.09 74.93 90)
+			(effects
+				(font
+					(size 1.27 1.27)
+				)
+				(hide yes)
+			)
+		)
 		(pin "1"
 		)
@@
 			(at 134.62 58.42 0)
 			(effects
+				(font
+					(size 1.27 1.27)
+				)
+				(hide yes)
+			)
+		)
+		(property "LCSC" "C98220"
+			(at 134.62 58.42 0)
+			(effects
