File: kicad/led_panel.kicad_sch (KiCad schematic)
At the start: 10 parts

Commit message: adjustments to design on kicad
Parts:
- APP_1, APP_2, APP_3: footprint (none) -> LED_SMD:LED_0805_2012Metric
- LAN1: renamed from LAN; footprint (none) -> LED_SMD:LED_0805_2012Metric
- PWR1: renamed from PWR; footprint (none) -> LED_SMD:LED_0805_2012Metric
- R10, R6, R7, R8, R9: value R -> 220; footprint (none) -> Resistor_SMD:R_0603_1608Metric
Changed lines of the file:
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@@
       (effects (font (size 1.27 1.27)) (justify right))
     )
-    (property "Footprint" "" (at 101.6 54.61 0)
+    (property "Footprint" "LED_SMD:LED_0805_2012Metric" (at 101.6 54.61 0)
       (effects (font (size 1.27 1.27)) hide)
     )
@@
   (symbol (lib_id "Device:LED") (at 63.5 54.61 90) (unit 1)
     (in_bom yes) (on_board yes) (dnp no) (fields_autoplaced)
-    (property "Reference" "LAN" (at 67.31 54.9275 90)
+    (property "Reference" "LAN1" (at 67.31 54.9275 90)
       (effects (font (size 1.27 1.27)) (justify right))
     )
@@
       (effects (font (size 1.27 1.27)) (justify right))
     )
-    (property "Footprint" "" (at 63.5 54.61 0)
+    (property "Footprint" "LED_SMD:LED_0805_2012Metric" (at 63.5 54.61 0)
       (effects (font (size 1.27 1.27)) hide)
     )
@@
       (project "project"
         (path "/9538e4ed-27e6-4c37-b989-9859dc0d49e8/b5459d7a-1bde-4bce-998a-859d3b17613f"
-          (reference "LAN") (unit 1)
+          (reference "LAN1") (unit 1)
         )
       )
@@
       (effects (font (size 1.27 1.27)) (justify left))
     )
-    (property "Value" "R" (at 53.34 48.26 0)
-      (effects (font (size 1.27 1.27)) (justify left))
-    )
-    (property "Footprint" "" (at 49.022 46.99 90)
+    (property "Value" "220" (at 53.34 48.26 0)
+      (effects (font (size 1.27 1.27)) (justify left))
+    )
+    (property "Footprint" "Resistor_SMD:R_0603_1608Metric" (at 49.022 46.99 90)
       (effects (font (size 1.27 1.27)) hide)
     )
@@
       (effects (font (size 1.27 1.27)) (justify right))
     )
-    (property "Footprint" "" (at 76.2 54.61 0)
+    (property "Footprint" "LED_SMD:LED_0805_2012Metric" (at 76.2 54.61 0)
       (effects (font (size 1.27 1.27)) hide)
     )
@@
       (effects (font (size 1.27 1.27)) (justify right))
     )
-    (property "Footprint" "" (at 88.9 54.61 0)
+    (property "Footprint" "LED_SMD:LED_0805_2012Metric" (at 88.9 54.61 0)
       (effects (font (size 1.27 1.27)) hide)
     )
@@
       (effects (font (size 1.27 1.27)) (justify left))
     )
-    (property "Value" "R" (at 78.74 48.26 0)
-      (effects (font (size 1.27 1.27)) (justify left))
-    )
-    (property "Footprint" "" (at 74.422 46.99 90)
+    (property "Value" "220" (at 78.74 48.26 0)
+      (effects (font (size 1.27 1.27)) (justify left))
+    )
+    (property "Footprint" "Resistor_SMD:R_0603_1608Metric" (at 74.422 46.99 90)
       (effects (font (size 1.27 1.27)) hide)
     )
@@
   (symbol (lib_id "Device:LED") (at 50.8 54.61 90) (unit 1)
     (in_bom yes) (on_board yes) (dnp no) (fields_autoplaced)
-    (property "Reference" "PWR" (at 54.61 54.9275 90)
+    (property "Reference" "PWR1" (at 54.61 54.9275 90)
       (effects (font (size 1.27 1.27)) (justify right))
     )
@@
       (effects (font (size 1.27 1.27)) (justify right))
     )
-    (property "Footprint" "" (at 50.8 54.61 0)
+    (property "Footprint" "LED_SMD:LED_0805_2012Metric" (at 50.8 54.61 0)
       (effects (font (size 1.27 1.27)) hide)
     )
@@
       (project "project"
         (path "/9538e4ed-27e6-4c37-b989-9859dc0d49e8/b5459d7a-1bde-4bce-998a-859d3b17613f"
-          (reference "PWR") (unit 1)
+          (reference "PWR1") (unit 1)
         )
       )
@@
       (effects (font (size 1.27 1.27)) (justify left))
     )
-    (property "Value" "R" (at 66.04 48.26 0)
-      (effects (font (size 1.27 1.27)) (justify left))
-    )
-    (property "Footprint" "" (at 61.722 46.99 90)
+    (property "Value" "220" (at 66.04 48.26 0)
+      (effects (font (size 1.27 1.27)) (justify left))
+    )
+    (property "Footprint" "Resistor_SMD:R_0603_1608Metric" (at 61.722 46.99 90)
       (effects (font (size 1.27 1.27)) hide)
     )
@@
       (effects (font (size 1.27 1.27)) (justify left))
     )
-    (property "Value" "R" (at 91.44 48.26 0)
-      (effects (font (size 1.27 1.27)) (justify left))
-    )
-    (property "Footprint" "" (at 87.122 46.99 90)
+    (property "Value" "220" (at 91.44 48.26 0)
+      (effects (font (size 1.27 1.27)) (justify left))
+    )
+    (property "Footprint" "Resistor_SMD:R_0603_1608Metric" (at 87.122 46.99 90)
       (effects (font (size 1.27 1.27)) hide)
     )
@@
       (effects (font (size 1.27 1.27)) (justify left))
     )
-    (property "Value" "R" (at 104.14 48.26 0)
-      (effects (font (size 1.27 1.27)) (justify left))
-    )
-    (property "Footprint" "" (at 99.822 46.99 90)
-      (effects (font (size 1.27 1.27)) hide)
-    )
+    (property "Value" "220" (at 104.14 48.26 0)
+      (effects (font (size 1.27 1.27)) (justify left))
+    )
+    (property "Footprint" "Resistor_SMD:R_0603_1608Metric" (at 99.822 46.99 90)
+      (effects (font (size 1.27 1.27)) hide)
+    )

Commit message: routed pcb, only bom left to do
Changed lines of the file:
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@@
 		(fields_autoplaced yes)
 		(property "Reference" "APP_3"
-			(at 105.41 54.9275 90)
+			(at 105.41 54.9274 90)
 			(effects
 				(font
@@
 		)
 		(property "Value" "LED"
-			(at 105.41 57.4675 90)
+			(at 105.41 57.4674 90)
 			(effects
 				(font
@@
 			)
 		)
-		(property "Description" ""
+		(property "Description" "Light emitting diode"
 			(at 101.6 54.61 0)
 			(effects
@@
 		(fields_autoplaced yes)
 		(property "Reference" "LAN1"
-			(at 67.31 54.9275 90)
+			(at 67.31 54.9274 90)
 			(effects
 				(font
@@
 		)
 		(property "Value" "LED"
-			(at 67.31 57.4675 90)
+			(at 67.31 57.4674 90)
 			(effects
 				(font
@@
 			)
 		)
-		(property "Description" ""
+		(property "Description" "Light emitting diode"
 			(at 63.5 54.61 0)
 			(effects
@@
 		(fields_autoplaced yes)
 		(property "Reference" "R6"
-			(at 53.34 45.72 0)
+			(at 53.34 45.7199 0)
 			(effects
 				(font
@@
 		)
 		(property "Value" "220"
-			(at 53.34 48.26 0)
+			(at 53.34 48.2599 0)
 			(effects
 				(font
@@
 			)
 		)
-		(property "Description" ""
+		(property "Description" "Resistor"
 			(at 50.8 46.99 0)
 			(effects
@@
 		(fields_autoplaced yes)
 		(property "Reference" "APP_1"
-			(at 80.01 54.9275 90)
+			(at 80.01 54.9274 90)
 			(effects
 				(font
@@
 		)
 		(property "Value" "LED"
-			(at 80.01 57.4675 90)
+			(at 80.01 57.4674 90)
 			(effects
 				(font
@@
 			)
 		)
-		(property "Description" ""
+		(property "Description" "Light emitting diode"
 			(at 76.2 54.61 0)
 			(effects
@@
 		(fields_autoplaced yes)
 		(property "Reference" "APP_2"
-			(at 92.71 54.9275 90)
+			(at 92.71 54.9274 90)
 			(effects
 				(font
@@
 		)
 		(property "Value" "LED"
-			(at 92.71 57.4675 90)
+			(at 92.71 57.4674 90)
 			(effects
 				(font
@@
 			)
 		)
-		(property "Description" ""
+		(property "Description" "Light emitting diode"
 			(at 88.9 54.61 0)
 			(effects
@@
 		(fields_autoplaced yes)
 		(property "Reference" "R8"
-			(at 78.74 45.72 0)
+			(at 78.74 45.7199 0)
 			(effects
 				(font
@@
 		)
 		(property "Value" "220"
-			(at 78.74 48.26 0)
+			(at 78.74 48.2599 0)
 			(effects
 				(font
@@
 			)
 		)
-		(property "Description" ""
+		(property "Description" "Resistor"
 			(at 76.2 46.99 0)
 			(effects
@@
 		(fields_autoplaced yes)
 		(property "Reference" "PWR1"
-			(at 54.61 54.9275 90)
+			(at 54.61 54.9274 90)
 			(effects
 				(font
@@
 		)
 		(property "Value" "LED"
-			(at 54.61 57.4675 90)
+			(at 54.61 57.4674 90)
 			(effects
 				(font
@@
 			)
 		)
-		(property "Description" ""
+		(property "Description" "Light emitting diode"
 			(at 50.8 54.61 0)
 			(effects
@@
 		(fields_autoplaced yes)
 		(property "Reference" "R7"
-			(at 66.04 45.72 0)
+			(at 66.04 45.7199 0)
 			(effects
 				(font
@@
 		)
 		(property "Value" "220"
-			(at 66.04 48.26 0)
+			(at 66.04 48.2599 0)
 			(effects
 				(font
@@
 			)
 		)
-		(property "Description" ""
+		(property "Description" "Resistor"
 			(at 63.5 46.99 0)
 			(effects
@@
 		(fields_autoplaced yes)
 		(property "Reference" "R9"
-			(at 91.44 45.72 0)
+			(at 91.44 45.7199 0)
 			(effects
 				(font
@@
 		)
 		(property "Value" "220"
-			(at 91.44 48.26 0)
+			(at 91.44 48.2599 0)
 			(effects
 				(font
@@
 			)
 		)
-		(property "Description" ""
+		(property "Description" "Resistor"
 			(at 88.9 46.99 0)
 			(effects
@@
 		(fields_autoplaced yes)
 		(property "Reference" "R10"
-			(at 104.14 45.72 0)
+			(at 104.14 45.7199 0)
 			(effects
 				(font
@@
 		)
 		(property "Value" "220"
-			(at 104.14 48.26 0)
+			(at 104.14 48.2599 0)
 			(effects
 				(font
@@
 			)
 		)
-		(property "Description" ""
+		(property "Description" "Resistor"
 			(at 101.6 46.99 0)
 			(effects
@@
 		)
 		(property "Value" "+3V3"
-			(at 50.8 33.02 0)
-			(effects
-				(font
-					(size 1.27 1.27)
-				)
+			(at 53.34 36.8299 0)
+			(effects
+				(font
+					(size 1.27 1.27)
+				)
+				(justify left)
 			)
 		)
@@
 			)
 		)
-		(property "Description" ""
+		(property "Description" "Power symbol creates a global label with name \"+3V3\""
 			(at 50.8 38.1 0)
 			(effects
@@
 		)
 		(property "Value" "GND"
-			(at 101.6 68.58 0)
-			(effects
-				(font
-					(size 1.27 1.27)
-				)
+			(at 104.14 64.7699 0)
+			(effects
+				(font
+					(size 1.27 1.27)
+				)
+				(justify left)
 			)
 		)
@@
 			)
 		)
-		(property "Description" ""
+		(property "Description" "Power symbol creates a global label with name \"GND\" , ground"
 			(at 101.6 63.5 0)
 			(effects

Commit message: kicad changes
Parts:
- APP_1, APP_2, APP_3, LAN1, PWR1: LCSC (none) -> C51933308
- R10, R6, R7, R8, R9: LCSC (none) -> C22962
Changed lines of the file:
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@@
+			)
+		)
+		(property "LCSC" "C51933308"
+			(at 101.6 54.61 90)
+			(effects
+				(font
+					(size 1.27 1.27)
+				)
+				(hide yes)
 			)
 		)
@@
 			)
 		)
+		(property "LCSC" "C51933308"
+			(at 63.5 54.61 90)
+			(effects
+				(font
+					(size 1.27 1.27)
+				)
+				(hide yes)
+			)
+		)
 		(pin "2"
 		)
@@
 			)
 		)
+		(property "LCSC" "C22962"
+			(at 50.8 46.99 0)
+			(effects
+				(font
+					(size 1.27 1.27)
+				)
+				(hide yes)
+			)
+		)
 		(pin "1"
 		)
@@
 			)
 		)
+		(property "LCSC" "C51933308"
+			(at 76.2 54.61 90)
+			(effects
+				(font
+					(size 1.27 1.27)
+				)
+				(hide yes)
+			)
+		)
 		(pin "2"
 		)
@@
 			)
 		)
+		(property "LCSC" "C51933308"
+			(at 88.9 54.61 90)
+			(effects
+				(font
+					(size 1.27 1.27)
+				)
+				(hide yes)
+			)
+		)
 		(pin "2"
 		)
@@
 			)
 		)
+		(property "LCSC" "C22962"
+			(at 76.2 46.99 0)
+			(effects
+				(font
+					(size 1.27 1.27)
+				)
+				(hide yes)
+			)
+		)
 		(pin "1"
 		)
@@
 			)
 		)
+		(property "LCSC" "C51933308"
+			(at 50.8 54.61 90)
+			(effects
+				(font
+					(size 1.27 1.27)
+				)
+				(hide yes)
+			)
+		)
 		(pin "2"
 		)
@@
 			)
 		)
+		(property "LCSC" "C22962"
+			(at 63.5 46.99 0)
+			(effects
+				(font
+					(size 1.27 1.27)
+				)
+				(hide yes)
+			)
+		)
 		(pin "1"
 		)
@@
 			)
 		)
+		(property "LCSC" "C22962"
+			(at 88.9 46.99 0)
+			(effects
+				(font
+					(size 1.27 1.27)
+				)
+				(hide yes)
+			)
+		)
 		(pin "1"
 		)
@@
 			(at 101.6 46.99 0)
 			(effects
+				(font
+					(size 1.27 1.27)
+				)
+				(hide yes)
+			)
+		)
+		(property "LCSC" "C22962"
+			(at 101.6 46.99 0)
+			(effects
